File: parts/extruder pcb/extruderevolved.kicad_pcb (KiCad board)
At the start: 2 copper layers, 68 x 57 mm, 8 parts, among them CN1 B-3102R24P-A000, CN2 HC-1.25-2PWT, CN3 HC-1.25-3PWT, CN4 HC-1.25-4PWT, CN5 HC-1.25-5PWT, CN6 X2011WRS-02A-9TSN, CN7 HC-1.25-2PWT, CN8 HC-1.25-2PWT

Commit message: Add files via upload
Routing:
- net Empty "DET" #1: track 0.00 -> 38.9 mm
- net Empty "DET" #2: track 0.00 -> 35.3 mm
- net Heater-: track 56.6 -> 65.3 mm, vias 1 -> 0
- net Heater+: track 50.2 -> 56.0 mm
- net Probe #2: track 59.6 -> 63.4 mm
- net GND: track 129.4 -> 132.9 mm
- net E Motor #3: track 43.8 -> 46.9 mm, vias 0 -> 1
- net E Motor #1: track 40.4 -> 43.0 mm
- net E Motor #2: track 43.7 -> 45.9 mm, vias 0 -> 1
- net Probe #4: track 57.7 -> 59.7 mm
- net Termistor-: track 56.6 -> 54.8 mm, vias 1 -> 0
- net Part Cooling Fan+: track 68.7 -> 66.9 mm, vias 0 -> 1
- net Part Cooling Fan-: track 60.2 -> 61.6 mm, vias 0 -> 1
- net Thermistor+: track 53.6 -> 52.4 mm, vias 1 -> 0
- net Fan-: track 34.7 -> 33.6 mm, vias 1 -> 0
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Other:
- board size 68 x 57 mm -> 67 x 57 mm
